File: yokan-tracker.kicad_pcb (KiCad board)
At the start: 2 copper layers, 40 x 25 mm, 3 parts, among them U1 XIAO_ESP32_C6, U2 LSM6DSV_Module

Commit message: fix
Parts:
- moved U2 5.00 mm to (35.0, 13.0)
- moved C1 2.00 mm to (24.0, 8.00)
Routing:
- net INT1: track 33.0 -> 0.00 mm
- net SCL: track 22.4 -> 0.00 mm
- net SDA: track 21.7 -> 0.00 mm
- net +3V3: track 6.96 -> 0.00 mm
- net GND: track 6.78 -> 0.00 mm
Other:
- board size 40 x 25 mm -> 50 x 25 mm
- board text added: "SlimeVR Tracker XIAO ESP32-C6 + LSM6DSV"
- board text added: "SlimeVR: internal I2C pull-ups / C1=100nF bypass / SDO->GND=0x6A / CS->VCC=I2C"
- board text removed: "SlimeVR Tracker XIAO ESP32-C6 + LSM6DSV 40mm x 25mm"
- board text removed: "SlimeVR: internal I2C pull-ups / C1=100nF bypass SDO(1)->GND=0x6A / CS(6)->VCC=I2C"
Changed lines of the file:
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@@
 	(layers
 		(0 "F.Cu" signal)
-		(31 "B.Cu" signal)
-		(32 "B.Adhes" user "B.Adhesive")
-		(33 "F.Adhes" user "F.Adhesive")
-		(34 "B.Paste" user)
-		(35 "F.Paste" user)
-		(36 "B.SilkS" user "B.Silkscreen")
-		(37 "F.SilkS" user "F.Silkscreen")
-		(38 "B.Mask" user)
-		(39 "F.Mask" user)
-		(40 "Dwgs.User" user "User.Drawings")
-		(41 "Cmts.User" user "User.Comments")
-		(42 "Eco1.User" user "User.Eco1")
-		(43 "Eco2.User" user "User.Eco2")
-		(44 "Edge.Cuts" user)
-		(45 "Margin" user)
-		(46 "B.CrtYd" user "B.Courtyard")
-		(47 "F.CrtYd" user "F.Courtyard")
-		(48 "B.Fab" user "B.Fabrication")
-		(49 "F.Fab" user "F.Fabrication")
-		(50 "User.1" user)
-		(51 "User.2" user)
-		(52 "User.3" user)
-		(53 "User.4" user)
-		(54 "User.5" user)
-		(55 "User.6" user)
-		(56 "User.7" user)
-		(57 "User.8" user)
-		(58 "User.9" user)
+		(2 "B.Cu" signal)
+		(9 "F.Adhes" user "F.Adhesive")
+		(11 "B.Adhes" user "B.Adhesive")
+		(13 "F.Paste" user)
+		(15 "B.Paste" user)
+		(5 "F.SilkS" user "F.Silkscreen")
+		(7 "B.SilkS" user "B.Silkscreen")
+		(1 "F.Mask" user)
+		(3 "B.Mask" user)
+		(17 "Dwgs.User" user "User.Drawings")
+		(19 "Cmts.User" user "User.Comments")
+		(21 "Eco1.User" user "User.Eco1")
+		(23 "Eco2.User" user "User.Eco2")
+		(25 "Edge.Cuts" user)
+		(27 "Margin" user)
+		(31 "F.CrtYd" user "F.Courtyard")
+		(29 "B.CrtYd" user "B.Courtyard")
+		(35 "F.Fab" user "F.Fabrication")
+		(33 "B.Fab" user "B.Fabrication")
 	)
 	(setup
@@
 		(allow_soldermask_bridges_in_footprints no)
 		(pcbplotparams
-			(layerselection 0x00010fc_ffffffff)
-			(plot_on_all_layers_selection 0x0000000_00000000)
+			(layerselection 0x00000000_00000000_000010fc_ffffffff)
+			(plot_on_all_layers_selection 0x00000000_00000000_00000000_00000000)
 			(disableapertmacros no)
 			(usegerberextensions no)
@@
 			(effects (font (size 1.27 1.27) (thickness 0.15)))
 		)
-		(net 5 "INT1")
-		(net 3 "SDA")
-		(net 4 "SCL")
-		(net 1 "+3V3")
-		(net 2 "GND")
 		(attr smd)
 		(fp_line (start 0 -1.987) (end 0 -19.132) (stroke (width 0.1) (type solid)) (layer "F.SilkS"))
@@
 	(footprint "yokan-tracker:LSM6DSV_Module"
 		(layer "F.Cu")
-		(at 30 13)
+		(at 35 13)
 		(property "Reference" "U2"
 			(at 0 -11 0)
@@
 		(pad "6" thru_hole circle (at -5.5 5.08) (size 1.6 1.6) (drill 0.8) (layers "*.Cu" "*.Mask") (net 1 "+3V3"))
 		(pad "7" thru_hole circle (at -5.5 7.62) (size 1.6 1.6) (drill 0.8) (layers "*.Cu" "*.Mask") (net 2 "GND"))
-		(pad "8" thru_hole circle (at 5.5 -5.08) (size 1.6 1.6) (drill 0.8) (layers "*.Cu" "*.Mask") (net 0 ""))
-		(pad "9" thru_hole circle (at 5.5 -2.54) (size 1.6 1.6) (drill 0.8) (layers "*.Cu" "*.Mask") (net 0 ""))
+		(pad "8" thru_hole circle (at 5.5 -5.08) (size 1.6 1.6) (drill 0.8) (layers "*.Cu" "*.Mask"))
+		(pad "9" thru_hole circle (at 5.5 -2.54) (size 1.6 1.6) (drill 0.8) (layers "*.Cu" "*.Mask"))
 		(pad "10" thru_hole circle (at 5.5 0) (size 1.6 1.6) (drill 0.8) (layers "*.Cu" "*.Mask") (net 5 "INT1"))
-		(pad "11" thru_hole circle (at 5.5 2.54) (size 1.6 1.6) (drill 0.8) (layers "*.Cu" "*.Mask") (net 0 ""))
-		(pad "12" thru_hole circle (at 5.5 5.08) (size 1.6 1.6) (drill 0.8) (layers "*.Cu" "*.Mask") (net 0 ""))
+		(pad "11" thru_hole circle (at 5.5 2.54) (size 1.6 1.6) (drill 0.8) (layers "*.Cu" "*.Mask"))
+		(pad "12" thru_hole circle (at 5.5 5.08) (size 1.6 1.6) (drill 0.8) (layers "*.Cu" "*.Mask"))
 	)
 	(footprint "Capacitor_SMD:C_0402_1005Metric"
 		(layer "F.Cu")
-		(at 22 8)
+		(at 24 8)
 		(property "Reference" "C1"
 			(at 0 -1.43 0)
@@
 	(gr_rect
 		(start 0 0)
-		(end 40 25)
+		(end 50 25)
 		(stroke (width 0.05) (type solid))
 		(fill no)
 		(layer "Edge.Cuts")
 	)
-	(gr_text "SlimeVR Tracker\nXIAO ESP32-C6 + LSM6DSV\n40mm x 25mm"
-		(at 20 26.5 0)
+	(gr_text "SlimeVR Tracker XIAO ESP32-C6 + LSM6DSV"
+		(at 1 26 0)
 		(layer "F.SilkS")
 		(effects (font (size 1 1) (thickness 0.15)) (justify left))
 	)
-	(gr_text "SlimeVR: internal I2C pull-ups / C1=100nF bypass\nSDO(1)->GND=0x6A / CS(6)->VCC=I2C"
+	(gr_text "SlimeVR: internal I2C pull-ups / C1=100nF bypass / SDO->GND=0x6A / CS->VCC=I2C"
 		(at 1 27.5 0)
 		(layer "Cmts.User")
-		(effects (font (size 1 1) (thickness 0.15)) (justify left))
-	)
-	(segment
-		(start 2.835 8.42)
-		(end 35.5 13)
-		(width 0.25)
-		(layer "F.Cu")
-		(net 5 "INT1")
-	)
-	(segment
-		(start 2.835 16.04)
-		(end 24.5 15.54)
-		(width 0.25)
-		(layer "F.Cu")
-		(net 3 "SDA")
-	)
-	(segment
-		(start 2.835 18.58)
-		(end 24.5 13)
-		(width 0.25)
-		(layer "F.Cu")
-		(net 4 "SCL")
-	)
-	(segment
-		(start 19 10.96)
-		(end 21.27 8)
-		(width 0.5)
-		(layer "F.Cu")
-		(net 1 "+3V3")
-	)
-	(segment
-		(start 21.27 8)
-		(end 24.5 7.92)
-		(width 0.5)
-		(layer "F.Cu")
-		(net 1 "+3V3")
-	)
-	(segment
-		(start 19 8.42)
-		(end 22.73 8)
-		(width 0.5)
-		(layer "F.Cu")
-		(net 2 "GND")
-	)
-	(segment
-		(start 22.73 8)
-		(end 24.5 10.46)
-		(width 0.5)
-		(layer "F.Cu")
-		(net 2 "GND")
+		(effects (font (size 0.8 0.8) (thickness 0.12)) (justify left))
 	)
 )

Commit message: バージョン対応
Parts:
- moved C1 155.6 mm to (149.5, 100.0)
- moved U1 155.6 mm to (127.5, 116.0)
- moved U2 155.6 mm to (160.5, 105.0)
